File: PCB-sch/PCB-sch.kicad_sch (KiCad schematic)
At the start: 20 parts, among them J1 AVR-ISP-6, SW1 SW_Push, U1 ATmega32U4-A

Commit message: test
Parts:
- removed C?: 0.1u, symbol Device:C_Small
- added R6: 10k, Resistor_SMD:R_0805_2012Metric_Pad1.20x1.40mm_HandSolder, symbol Device:R_Small
- C1, C2, C3, C5, C6, C7, C8: renamed from C?; footprint (none) -> Capacitor_SMD:C_0805_2012Metric_Pad1.18x1.45mm_HandSolder
- F1: renamed from F?; footprint (none) -> Fuse:Fuse_1206_3216Metric_Pad1.42x1.75mm_HandSolder
- J1: footprint (none) -> random-keyboard-parts:Reset_Pretty-Mask
- R1, R2, R3, R4, R5: renamed from R?; footprint (none) -> Resistor_SMD:R_0805_2012Metric_Pad1.20x1.40mm_HandSolder
- SW1: footprint (none) -> Button_Switch_SMD:SW_SPST_SKQG_WithStem
- U2: renamed from U?; footprint (none) -> random-keyboard-parts:SOT143B
- USB1: renamed from USB?; footprint (none) -> Type-C:HRO-TYPE-C-31-M-12-HandSoldering
- Y1: renamed from Y?; footprint (none) -> Crystal:Crystal_SMD_3225-4Pin_3.2x2.5mm_HandSoldering
Connections:
- net +5V: now also R6.1
- net RESET: now also R6.2
- net DP: now reaches R3.1, U2.2 (IO1), USB1.6 (DP1), USB1.8 (DP2)
- net DN: now reaches R2.1, U2.3 (IO2), USB1.5 (DN2), USB1.7 (DN1)
- net row0: now reaches U1.1 (PE6)
- net col8: now reaches U1.19 (PD1)
- net col9: now reaches U1.20 (PD2)
- net col10: now reaches U1.21 (PD3)
- net col11: now reaches U1.22 (PD5)
- net col12: now reaches U1.25 (PD4)
- net col13: now reaches U1.26 (PD6)
- net col0: now reaches U1.28 (PB4)
- net col1: now reaches U1.29 (PB5)
- net col2: now reaches U1.30 (PB6)
- net col3: now reaches U1.31 (PC6)
- net col4: now reaches U1.32 (PC7)
- net row4: now reaches U1.36 (PF7)
- net col5: now reaches U1.37 (PF6)
- net col6: now reaches U1.38 (PF5)
- net row1: now reaches U1.39 (PF4)
- net row3: now reaches U1.40 (PF1)
- net row2: now reaches U1.41 (PF0)
- net col7: now reaches U1.8 (PB0)
- no-connect marks 3 -> 6
Other:
- moved on the sheet: C5
