File: PCB-sch/matrix.sch.kicad_sch (KiCad schematic)
At the start: 122 parts

Commit message: test
Parts:
- D1, D10, D11, D12, D13, D14, D15, D16, D17, D18, D19, D2, D20, D21, D22, D23, D24, D25, D26, D27, D28, D29, D3, D30, D31, D32, D33, D34, D35, D36, D37, D38, D39, D4, D40, D41, D42, D43, D44, D45, D46, D47, D48, D49, D5, D50, D51, D52, D53, D54, D55, D56, D57, D58, D59, D6, D60, D61, D7, D8, D9: footprint (none) -> Diode_SMD:D_SOD-123
- K?1, K?10, K?11, K?12, K?13, K?16, K?17, K?18, K?19, K?2, K?20, K?21, K?22, K?23, K?24, K?25, K?26, K?27, K?3, K?30, K?31, K?32, K?33, K?34, K?35, K?36, K?37, K?38, K?39, K?40, K?43, K?44, K?45, K?46, K?47, K?48, K?49, K?5, K?50, K?51, K?52, K?6, K?7, K?8, K?9: footprint (none) -> MX_Hotswap:MX-Hotswap-1U
- K?14: footprint (none) -> MX_Hotswap:MX-Hotswap-2U
- K?15, K?28: footprint (none) -> MX_Hotswap:MX-Hotswap-1.5U
- K?29: footprint (none) -> MX_Hotswap:MX-Hotswap-1.75U
- K?4: value #2 -> #3; footprint (none) -> MX_Hotswap:MX-Hotswap-1U
- K?41, K?42: footprint (none) -> MX_Hotswap:MX-Hotswap-2.25U
- K?53: footprint (none) -> MX_Hotswap:MX-Hotswap-2.75U
- K?54, K?55, K?56, K?58, K?59, K?60, K?61: footprint (none) -> MX_Hotswap:MX-Hotswap-1.25U
- K?57: footprint (none) -> MX_Hotswap:MX-Hotswap-6.25U-ReversedStabilizers
Connections:
- net col9: now reaches K?10.2, K?24.2, K?38.2, K?51.2
- net col11: now reaches K?12.2, K?26.2, K?40.2, K?59.2
- net col3: now reaches K?18.2, K?32.2, K?4.2, K?45.2
- net col10: now reaches K?11.2, K?25.2, K?39.2, K?52.2, K?58.2
- net col7: now reaches K?22.2, K?36.2, K?49.2, K?8.2
- net col2: now reaches K?17.2, K?3.2, K?31.2, K?44.2, K?56.2
- net col4: now reaches K?19.2, K?33.2, K?46.2, K?5.2
- net col6: now reaches K?21.2, K?35.2, K?48.2, K?57.2, K?7.2
- net col13: now reaches K?14.2, K?28.2, K?41.2, K?53.2, K?61.2
- net col1: now reaches K?16.2, K?2.2, K?30.2, K?43.2, K?55.2
- net col12: now reaches K?13.2, K?27.2, K?60.2
- net col0: now reaches K?1.2, K?15.2, K?29.2, K?42.2, K?54.2
- net col5: now reaches K?20.2, K?34.2, K?47.2, K?6.2
- net col8: now reaches K?23.2, K?37.2, K?50.2, K?9.2
Other:
- moved on the sheet: D1, D10, D11, D12, D13, D14, D15, D16, D17, D18, D19, D2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
